File: hardware/eagle/Linefollower_Bluepill.brd (EAGLE design)
At the start: 85 x 50 mm, 33 parts, among them CON1 EH_B8B-EH, IC1 LM1117IMPX-5.0, IC3 LM1117IMPX-3.3

Commit message: Removed Vin to VBat
Removed wrong connection to bluepill. It caused the blue pill's magic smoke to escape. Resolves #4
Connections:
- net V+: no longer U$1.P$40
Routing:
- net LIR: track 87.3 -> 88.8 mm
Other:
- board text added: "Robot-SM 2019 Line follower CASE Board 18/19 Rev. 1.2 Blue pill 2019-04-06"
- board text removed: "Robot-SM 2019 Line follower CASE Board 18/19 Rev. 1.1 Blue pill 2019-03-20"
Changed lines of the file:
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@@
 Line follower
 CASE Board 18/19
-Rev. 1.1 Blue pill
-2019-03-20
+Rev. 1.2 Blue pill
+2019-04-06
 </text>
 <text x="1.947721875" y="23.965459375" size="1.016" layer="27" rot="R90">Gnd</text>
@@
 <contactref element="RLED3" pad="2"/>
 <contactref element="R4" pad="1"/>
-<contactref element="U$1" pad="P$40"/>
 <contactref element="IC1" pad="3"/>
 <contactref element="C2" pad="1"/>
@@
 <wire x1="34.25" y1="33.75" x2="34.35640625" y2="33.825815625" width="0.889" layer="16"/>
 <wire x1="31.25" y1="29.5" x2="31.039" y2="29.439" width="0.889" layer="16"/>
-<wire x1="16.75" y1="29.25" x2="16.75" y2="24.25" width="0.889" layer="16"/>
-<wire x1="30.75" y1="29.25" x2="16.75" y2="29.25" width="0.889" layer="16"/>
-<wire x1="16.75" y1="24.25" x2="16.51" y2="24.13" width="0.889" layer="16"/>
+<wire x1="16.75" y1="29.25" x2="30.75" y2="29.25" width="0.889" layer="16"/>
 <wire x1="30.75" y1="29.25" x2="31.039" y2="29.439" width="0.889" layer="16"/>
 <wire x1="67.25" y1="21" x2="66.75" y2="20.5" width="0.889" layer="16"/>
@@
 <wire x1="16.256" y1="9.2456" x2="31.3944" y2="9.2456" width="0.889" layer="16"/>
 <wire x1="14.6558" y1="10.8458" x2="16.256" y2="9.2456" width="0.889" layer="16"/>
-<wire x1="14.6304" y1="22.1488" x2="16.256" y2="23.7744" width="0.889" layer="16"/>
-<wire x1="16.256" y1="23.7744" x2="16.51" y2="24.13" width="0.889" layer="16"/>
 <wire x1="14.6558" y1="22.1234" x2="14.6304" y2="22.1488" width="0.889" layer="16"/>
 <wire x1="14.6558" y1="10.8458" x2="14.6558" y2="11.93715625" width="0.889" layer="16"/>
@@
 <wire x1="14.2875" y1="12.30545625" x2="14.2875" y2="15.12654375" width="0.889" layer="16"/>
 <wire x1="14.2875" y1="15.12654375" x2="14.6558" y2="15.49484375" width="0.889" layer="16"/>
-<wire x1="14.6558" y1="15.49484375" x2="14.6558" y2="22.1234" width="0.889" layer="16"/>
+<wire x1="14.6558" y1="15.49484375" x2="14.6558" y2="21.59" width="0.889" layer="16"/>
 <contactref element="IC3" pad="3"/>
+<wire x1="14.6558" y1="21.59" x2="14.6558" y2="22.1234" width="0.889" layer="16"/>
 <wire x1="31.3944" y1="10.3632" x2="29.4138" y2="10.3632" width="0.889" layer="16"/>
 <wire x1="29.4138" y1="10.3632" x2="29.134" y2="10.643" width="0.889" layer="16"/>
+<wire x1="14.6558" y1="22.1234" x2="14.6558" y2="27.1558" width="0.889" layer="16"/>
+<wire x1="14.6558" y1="27.1558" x2="16.75" y2="29.25" width="0.889" layer="16"/>
 </signal>
 <signal name="LENCB">
@@
 <wire x1="62" y1="39.25" x2="62.23" y2="39.37" width="0.254" layer="1"/>
 <wire x1="30.5" y1="45.25" x2="30.42525625" y2="45.3058" width="0.254" layer="1"/>
-<wire x1="15.25" y1="24.25" x2="7.75" y2="16.75" width="0.254" layer="16"/>
-<wire x1="15.25" y1="34.5" x2="15.25" y2="24.25" width="0.254" layer="16"/>
-<wire x1="25" y1="34.5" x2="15.25" y2="34.5" width="0.254" layer="16"/>
+<wire x1="12.71" y1="21.71" x2="7.75" y2="16.75" width="0.254" layer="16"/>
+<wire x1="12.71" y1="34.5" x2="12.71" y2="21.71" width="0.254" layer="16"/>
+<wire x1="25" y1="34.5" x2="12.71" y2="34.5" width="0.254" layer="16"/>
 <wire x1="25.5" y1="35" x2="25" y2="34.5" width="0.254" layer="1"/>
 <wire x1="25.5" y1="40.5" x2="25.5" y2="35" width="0.254" layer="1"/>
